File: elec/layout/default/mpu6050.kicad_pcb (KiCad board)
At the start: 2 copper layers, 225.7 x 100.8 mm, 0 parts

Commit message: update layout
Parts:
- added C1: 16V 100nF X7R ±10% 0402 Multilayer Ceramic Capacitors MLCC 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, lib:C0402, F.Cu at (161.7, 87.3)
- added C2: 50V 2.2nF X7R ±10% 0603 Multilayer Ceramic Capacitors MLCC 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, lib:C0603, F.Cu at (153.9, 86.6)
- added R1: 62.5mW Thick Film Resistors ±100ppm/℃ ±1% 10kΩ 0402 Chip Re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, lib:R0402, F.Cu at (161.3, 85.7)
- added R2: 62.5mW Thick Film Resistors ±100ppm/℃ ±1% 10kΩ 0402 Chip Re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, lib:R0402, F.Cu at (154.2, 89.7)
- added R3: 62.5mW Thick Film Resistors ±100ppm/℃ ±1% 10kΩ 0402 Chip Re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, lib:R0402, F.Cu at (154.1, 88.7)
- added U1: , lib:QFN-24_L4.0-W4.0-P0.50-BL-EP2.7, F.Cu at (158.0, 87.7)
Routing:
- net gnd-1: track 0.00 -> 16.6 mm, vias 0 -> 2
- net vcc: track 0.00 -> 7.45 mm, vias 0 -> 3
- net sda: track 0.00 -> 1.70 mm
- net cpout: track 0.00 -> 1.45 mm
- net scl: track 0.00 -> 1.44 mm
- net interrupt: track 0.00 -> 1.30 mm
- net regout: track 0.00 -> 1.25 mm
